File: CM4_NAS.kicad_pcb (KiCad board)
At the start: 4 copper layers, 88.5 x 72.5 mm, 32 parts, among them J1 USB_A, J10 Conn_02x07_Odd_Even, J11 Conn_01x03, J12 Conn_01x03, J13 Conn_02x06_Odd_Even, J15 Temp_Sensor, J2 HDMI_header, J3 PCIe_conn, J4 Sata_PWR, J5 PWR_IN, J6 12-3.3_BUCK, J7 Fan_conn, J8 OLED_conn, J9 Conn_01x03, U1 74LVC1G07SE-7, U2 TPD4EUSB30, U3 TPD4EUSB30, U4 MagJack-0826-1G1T-43-F, U5 TPD4EUSB30, U6 EMC2301-1-ACZL-TR, U7 74LVC1G07SE-7

Commit message: Updated to Version 1.5, imported power circuitry for 12V input only
Parts:
- removed J5: PWR_IN, Connector_JST:JST_XH_B3B-XH-A_1x03_P2.50mm_Vertical
- removed J6: 12-3.3_BUCK, Connector_PinSocket_2.54mm:PinSocket_1x06_P2.54mm_Vertical
- removed U4: MagJack-0826-1G1T-43-F, CM4:MagJack_0826-1G1T-43-F
- added C10: 10u 35v, Capacitor_SMD:C_0805_2012Metric, F.Cu at (81.3, 111.8)
- added C11: 10u 35v, Capacitor_SMD:C_0805_2012Metric, F.Cu at (78.8, 90.7)
- added C12: 10u 35v, Capacitor_SMD:C_0805_2012Metric, F.Cu at (81.3, 114.4)
- added C13: 10u 35v, Capacitor_SMD:C_0805_2012Metric, F.Cu at (78.8, 88.6)
- added C14: 100n, Capacitor_SMD:C_0402_1005Metric, F.Cu at (77.8, 125.2)
- added C15: 10u 35v, Capacitor_SMD:C_0805_2012Metric, F.Cu at (81.3, 116.9)
- added C16: 10u 35v, Capacitor_SMD:C_0805_2012Metric, F.Cu at (78.8, 92.7)
- added C17: 100n, Capacitor_SMD:C_0402_1005Metric, F.Cu at (74.8, 109.3)
- added C18: 100n, Capacitor_SMD:C_0402_1005Metric, F.Cu at (72.4, 86.4)
- added C19: 100n, Capacitor_SMD:C_0402_1005Metric, F.Cu at (82.7, 109.8)
- added C20: 10u 35v, Capacitor_SMD:C_0805_2012Metric, F.Cu at (75.9, 125.6)
- added C21: 100n, Capacitor_SMD:C_0402_1005Metric, F.Cu at (81.3, 86.4)
- added C22: nf, Capacitor_SMD:C_0402_1005Metric, F.Cu at (79.4, 99.5)
- added C23: nf, Capacitor_SMD:C_0402_1005Metric, F.Cu at (84.6, 85.3)
- added C24: 1.2nF, Capacitor_SMD:C_0402_1005Metric, F.Cu at (83.8, 98.9)
- added C25: 1.2nF, Capacitor_SMD:C_0402_1005Metric, F.Cu at (84.7, 89.8)
- added C26: nf, Capacitor_SMD:C_0402_1005Metric, F.Cu at (92.0, 107.4)
- added C27: nf, Capacitor_SMD:C_0402_1005Metric, F.Cu at (83.8, 81.3)
- added C28: 10u, Capacitor_SMD:C_0805_2012Metric, F.Cu at (83.9, 71.3)
- added C29: 10u, Capacitor_SMD:C_0805_2012Metric, F.Cu at (103.2, 114.3)
- added C3: 10u 35v, Capacitor_SMD:C_0805_2012Metric, F.Cu at (73.7, 88.4)
- added C30: 10u, Capacitor_SMD:C_0805_2012Metric, F.Cu at (80.8, 77.9)
- added C31: 10u, Capacitor_SMD:C_0805_2012Metric, F.Cu at (103.2, 116.4)
- added C32: 10u, Capacitor_SMD:C_0805_2012Metric, F.Cu at (81.5, 71.2)
- added C33: 10u, Capacitor_SMD:C_0805_2012Metric, F.Cu at (95.8, 109.2)
- added C34: 10u, Capacitor_SMD:C_0805_2012Metric, F.Cu at (82.9, 77.9)
- added C35: 10u, Capacitor_SMD:C_0805_2012Metric, F.Cu at (97.9, 109.2)
- added C36: 100uF, Capacitor_Tantalum_SMD:CP_EIA-7343-31_Kemet-D, F.Cu at (88.4, 74.7)
- added C37: 100uF, Capacitor_Tantalum_SMD:CP_EIA-7343-31_Kemet-D, F.Cu at (96.5, 116.8)
- added C4: 10u 35v, Capacitor_SMD:C_0805_2012Metric, F.Cu at (76.2, 116.9)
- added C5: 100n 100v, Capacitor_SMD:C_0402_1005Metric, F.Cu at (89.9, 127.0)
- added C6: 10u 35v, Capacitor_SMD:C_0805_2012Metric, F.Cu at (73.7, 90.6)
- added C7: 10u 35v, Capacitor_SMD:C_0805_2012Metric, F.Cu at (76.2, 114.4)
- added C8: 10u 35v, Capacitor_SMD:C_0805_2012Metric, F.Cu at (76.2, 111.8)
- added C9: 10u 35v, Capacitor_SMD:C_0805_2012Metric, F.Cu at (73.7, 92.7)
- added D3: MMBZ5242BLT3G, Diode_SMD:D_SOT-23_ANK, F.Cu at (80.4, 125.9)
- added J0: ARJM11C7-502-AB-ER2-T, CM4:ABRACON_ARJM11C7-502-AB-ER2-T, F.Cu at (167.0, 131.5)
- added J14: Barrel_Jack, CM4:BarrelJack_Horizontal, F.Cu at (86.4, 129.5)
- added L1: SRN6045TA-3R3Y, Inductor_SMD:L_Bourns_SRN6045TA, F.Cu at (88.5, 111.8)
- added L2: SRN6045TA-3R3Y, Inductor_SMD:L_Bourns_SRN6045TA, F.Cu at (76.2, 73.7)
- added Q1: DMP3013SFV-7, Package_SON:Diodes_PowerDI3333-8, F.Cu at (84.8, 124.5)
- added R10: 20K 1%, Resistor_SMD:R_0402_1005Metric, F.Cu at (81.3, 98.9)
- added R11: 12K 1%, Resistor_SMD:R_0402_1005Metric, F.Cu at (84.6, 86.9)
- added R12: 12K 1%, Resistor_SMD:R_0402_1005Metric, F.Cu at (92.0, 105.6)
- added R13: 2.2K 1%, Resistor_SMD:R_0402_1005Metric, F.Cu at (83.8, 107.2)
- added R14: 47K 1%, Resistor_SMD:R_0402_1005Metric, F.Cu at (83.0, 80.2)
- added R15: 15K 1%, Resistor_SMD:R_0402_1005Metric, F.Cu at (81.2, 82.7)
- added R7: 12K 1%, Resistor_SMD:R_0402_1005Metric, F.Cu at (80.3, 128.8)
- added R8: 10R, Resistor_SMD:R_0402_1005Metric, F.Cu at (74.3, 106.1)
- added R9: 10R, Resistor_SMD:R_0402_1005Metric, F.Cu at (72.4, 83.8)
- added TP1: TestPoint, TestPoint:TestPoint_Pad_2.0x2.0mm, B.Cu at (81.3, 119.4)
- added TP2: TestPoint, TestPoint:TestPoint_Pad_2.0x2.0mm, B.Cu at (100.7, 112.8)
- added TP3: TestPoint, TestPoint:TestPoint_Pad_2.0x2.0mm, B.Cu at (96.5, 132.1)
- added TP4: TestPoint, TestPoint:TestPoint_Pad_2.0x2.0mm, B.Cu at (86.4, 94.0)
- added U8: AP64501SP-13, CM4:SOIC-8-1EP_3.9x4.9mm_P1.27mm_EP2.95x4.9mm_Mask2.71x3.4mm_ThermalVias, F.Cu at (78.7, 106.7)
- added U9: AP64501SP-13, CM4:SOIC-8-1EP_3.9x4.9mm_P1.27mm_EP2.95x4.9mm_Mask2.71x3.4mm_ThermalVias, F.Cu at (76.2, 83.8)
- R1, R2, R3, R4, R5, R6: footprint Resistor_THT:R_Axial_DIN0207_L6.3mm_D2.5mm_P7.62mm_Horizontal -> Resistor_SMD:R_0402_1005Metric
- moved R5 7.34 mm to (102.3, 129.3)
- moved R3 3.69 mm to (168.5, 103.5)
- moved R6 3.25 mm to (172.0, 72.8)
- moved U6 2.10 mm to (107.1, 127.8)
- moved C2 1.72 mm to (103.3, 135.1)
- moved R1 0.79 mm to (161.0, 99.0), turned to 180 degrees
- moved R4 0.49 mm to (170.0, 97.0), turned to -90 degrees
Connections:
- J2 pad 14: Net-(J2-Pad14) -> unconnected-(J2-UTILITY/HEAC+-Pad14)
- J3 pad A1: Net-(J3-PadA1) -> unconnected-(J3-nPRSNT1-PadA1)
- J3 pad A7: Net-(J3-PadA7) -> unconnected-(J3-TD0-PadA7)
- J3 pad B11: Net-(J3-PadB11) -> unconnected-(J3-nWAKE-PadB11)
- J3 pad B17: Net-(J3-PadB17) -> unconnected-(J3-nPRSNT2-PadB17)
- J3 pad B5: Net-(J3-PadB5) -> unconnected-(J3-SMCLK-PadB5)
- J3 pad B6: Net-(J3-PadB6) -> unconnected-(J3-SMDAT-PadB6)
- Module1 pad 104: Net-(Module1-Pad104) -> unconnected-(Module1B-Reserved-Pad104)
- Module1 pad 106: Net-(Module1-Pad106) -> unconnected-(Module1B-Reserved-Pad106)
- Module1 pad 19: Net-(Module1-Pad19) -> unconnected-(Module1A-Ethernet_nLED1(3.3v)-Pad19)
- Module1 pad 64: Net-(Module1-Pad64) -> unconnected-(Module1A-SD_DAT5-Pad64)
- Module1 pad 68: Net-(Module1-Pad68) -> unconnected-(Module1A-SD_DAT4-Pad68)
- Module1 pad 70: Net-(Module1-Pad70) -> unconnected-(Module1A-SD_DAT7-Pad70)
- Module1 pad 72: Net-(Module1-Pad72) -> unconnected-(Module1A-SD_DAT6-Pad72)
- Module1 pad 73: Net-(Module1-Pad73) -> unconnected-(Module1A-SD_VDD_Override-Pad73)
- U6 pad 7: Net-(U6-Pad7) -> unconnected-(U6-CLK-Pad7)
- U6 pad 8: Net-(U6-Pad8) -> unconnected-(U6-nALERT-Pad8)
Routing:
- net /+12v: track 0.00 -> 279.5 mm, vias 0 -> 8
- net +12V: track 151.3 -> 0.00 mm, vias 6 -> 0
- net /+3.3v: track 271.7 -> 370.7 mm, vias 6 -> 8
- net +3V3: track 82.2 -> 0.00 mm
- net Net-(J0-LED-L_K_GRN): track 7.02 -> 45.2 mm, vias 0 -> 2
- net Net-(J0-LED-R_K_YLW): track 4.45 -> 41.0 mm, vias 0 -> 1
- net Net-(U8-SW): track 0.00 -> 28.1 mm, vias 0 -> 6
- net +5V: track 237.7 -> 260.4 mm, vias 8 -> 12
- net GND: track 19.8 -> 41.6 mm, vias 66 -> 92
- net Net-(U9-COMP): track 0.00 -> 18.1 mm, vias 0 -> 2
- net Net-(U8-FB): track 0.00 -> 13.6 mm
- net /TRD0_N: track 20.0 -> 33.0 mm
- net Net-(U9-SW): track 0.00 -> 11.9 mm
- net /TRD0_P: track 20.0 -> 31.2 mm
- net /TRD3_P: track 23.4 -> 34.5 mm, vias 0 -> 2
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Other:
- board size 88.5 x 72.5 mm -> 108.6 x 72.5 mm
- board text added: "Ethernet"
- board text added: "RPi CM4 NAS rev1.5 by Koyami"
- board text removed: "3V3_BUCK"
- board text removed: "MagJack"
- board text removed: "PWR_IN"
- board text removed: "RPi CM4 NAS rev1.4"
